File: hardware/wifi-adapter/esp-wifi-adapter.sch (KiCad schematic (older format))
At the start: 10 parts

Commit message: WiFi adaptor schematics at v0.9
Parts:
- removed U?: MCP1826S, symbol MCP1826S
- added J3: CONN_01X06, Socket_Strips:Socket_Strip_Straight_1x06_Pitch2.54mm, symbol CONN_01X06
- added U1: MCP1826S, TO_SOT_Packages_SMD:SOT-223, symbol MCP1826S
- J1: renamed from J?; footprint (none) -> Socket_Strips:Socket_Strip_Straight_2x04_Pitch2.54mm
- J2: renamed from J?; footprint (none) -> Socket_Strips:Socket_Strip_Straight_2x05_Pitch2.54mm
- R1, R2, R3, R4, R5: renamed from R?; value R -> 10K; footprint (none) -> Resistors_SMD:R_1206_HandSoldering
- gave numbers to parts that had none: 2
Connections:
- net +3V3: now reaches Q1.1 (G)
- net +3V3: now also J1.1 (P1), J1.3 (P3), Q2.1 (G), R1.1, R2.1, R3.1, U1.3 (Vout)
- net at Q1.2 (S): now also J1.2 (P2), R2.2
- net at Q1.3 (D): now also J2.2 (P2), R4.2, J3.5 (P5)
- net at R3.2: now also J1.7 (P7), Q2.2 (S)
- net +5V: now reaches R4.1
- net +5V: now also J2.3 (P3), R5.1, J3.3 (P3), U1.1 (Vin)
- net at R5.2: now also J2.9 (P9), Q2.3 (D), J3.4 (P4)
- net at J1.5 (P5): now also R1.2
- net GND: now reaches J1.6 (P6)
- net GND: now also J1.8 (P8), J2.1 (P1), J3.1 (P1), U1.2 (GND)
Other:
- moved on the sheet: J1, J2, Q1, Q2, R1, R2, R3, R4, R5
